File: Hardware/Placa_PCB/Ground_Station.kicad_sch (KiCad schematic)
At the start: 0 parts

Commit message: Agregando el PCB terminado
Other:
- company: (none) -> FIUNA
- title: (none) -> Esquematico del Ground Station - IIS
Changed lines of the file:
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@@
 	(generator_version "9.0")
 	(paper "A4")
+	(title_block
+		(title "Esquematico del Ground Station - IIS")
+		(date "2026-03-20")
+		(company "FIUNA")
+		(comment 1 "Esteban Ruiz")
+		(comment 2 "Jose Medina")
+	)
 	(wire
 		(pts
