File: Hardware/Placa_PCB/MCU.kicad_sch (KiCad schematic)
At the start: 20 parts, among them J2 Conn_01x08_Pin, J3 Conn_01x08_Pin, SW1 RESET, SW2 BOOT, U2 ESP32-S3-WROOM-1, U4 MIC29302AWD

Commit message: Agregando el PCB terminado
Connections:
- net +3.3V: now also J3.3 (Pin_3), J3.4 (Pin_4), R5.1; no longer J2.3 (Pin_3)
- net +5V: now also J3.1 (Pin_1), J3.2 (Pin_2); no longer J2.2 (Pin_2), R5.1
- net 21 - LED: now also J2.8 (Pin_8); no longer J3.6 (Pin_6)
- net 3: now also J2.2 (Pin_2); no longer J2.4 (Pin_4)
- net 4: now also J2.3 (Pin_3); no longer J2.5 (Pin_5)
- net 5: now also J2.4 (Pin_4); no longer J2.6 (Pin_6)
- net 6: now also J2.5 (Pin_5); no longer J2.7 (Pin_7)
- net 7: now also J2.6 (Pin_6); no longer J2.8 (Pin_8)
- net 8: now also J2.7 (Pin_7); no longer J3.1 (Pin_1)
- net GNDD: now also J3.5 (Pin_5), J3.6 (Pin_6)
- net 15: no longer names the net of U2.8 (IO15)
- net 15: no longer J3.2 (Pin_2)
- net 16: no longer names the net of U2.9 (IO16)
- net 16: no longer J3.3 (Pin_3)
- net 17: no longer names the net of U2.10 (IO17)
- net 17: no longer J3.4 (Pin_4)
- net 18: no longer names the net of U2.11 (IO18)
- net 18: no longer J3.5 (Pin_5)
- no-connect marks 14 -> 18
Other:
- moved on the sheet: J2, J3
