File: Hardware/Placa_PCB/Alimentacion_USB.kicad_sch (KiCad schematic)
At the start: 7 parts, among them J1 USB_C_Receptacle_USB2.0_16P, U3 USBLC6-2SC6

Commit message: Agregando el PCB terminado
Connections:
- net D+: now also U3.3 (I/O2); no longer U3.4 (I/O2)
- net D-: now also U3.1 (I/O1); no longer U3.6 (I/O1)
- net USB_D+: now also U3.4 (I/O2); no longer U3.3 (I/O2)
- net USB_D-: now also U3.6 (I/O1); no longer U3.1 (I/O1)
Other:
- moved on the sheet: U3
Changed lines of the file:
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@@
 	(wire
 		(pts
-			(xy 180.34 91.44) (xy 184.15 91.44)
+			(xy 184.15 91.44) (xy 187.96 91.44)
 		)
 		(stroke
@@
 	(wire
 		(pts
-			(xy 189.23 81.28) (xy 189.23 86.36)
+			(xy 193.04 81.28) (xy 193.04 86.36)
 		)
 		(stroke
@@
 	(wire
 		(pts
-			(xy 189.23 99.06) (xy 189.23 102.87)
+			(xy 193.04 99.06) (xy 193.04 102.87)
 		)
 		(stroke
@@
 	(wire
 		(pts
-			(xy 194.31 91.44) (xy 195.58 91.44)
+			(xy 198.12 91.44) (xy 199.39 91.44)
 		)
 		(stroke
@@
 	(wire
 		(pts
-			(xy 194.31 93.98) (xy 195.58 93.98)
+			(xy 198.12 93.98) (xy 199.39 93.98)
 		)
 		(stroke
@@
 	(wire
 		(pts
-			(xy 180.34 93.98) (xy 184.15 93.98)
+			(xy 184.15 93.98) (xy 187.96 93.98)
 		)
 		(stroke
@@
 	)
 	(label "D-"
-		(at 180.34 91.44 180)
+		(at 199.39 91.44 0)
 		(effects
 			(font
 				(size 1.27 1.27)
 			)
-			(justify right bottom)
+			(justify left bottom)
 		)
 	)
 	(label "D+"
-		(at 180.34 93.98 180)
+		(at 199.39 93.98 0)
 		(effects
 			(font
 				(size 1.27 1.27)
 			)
-			(justify right bottom)
+			(justify left bottom)
 		)
 	)
 	(hierarchical_label "USB_D-"
 		(shape output)
-		(at 195.58 91.44 0)
+		(at 184.15 91.44 180)
 		(effects
 			(font
 				(size 1.27 1.27)
 			)
-			(justify left)
+			(justify right)
 		)
 	)
 	(hierarchical_label "USB_D+"
 		(shape output)
-		(at 195.58 93.98 0)
+		(at 184.15 93.98 180)
 		(effects
 			(font
 				(size 1.27 1.27)
 			)
-			(justify left)
+			(justify right)
 		)
 	)
@@
 	(symbol
 		(lib_id "power:GNDD")
-		(at 189.23 102.87 0)
+		(at 193.04 102.87 0)
 		(unit 1)
 		(exclude_from_sim no)
@@
 		(fields_autoplaced yes)
 		(property "Reference" "#PWR05"
-			(at 189.23 109.22 0)
+			(at 193.04 109.22 0)
 			(effects
 				(font
@@
 		)
 		(property "Value" "GNDD"
-			(at 189.23 106.68 0)
+			(at 193.04 106.68 0)
 			(effects
 				(font
@@
 		)
 		(property "Footprint" ""
-			(at 189.23 102.87 0)
+			(at 193.04 102.87 0)
 			(effects
 				(font
@@
 		)
 		(property "Datasheet" ""
-			(at 189.23 102.87 0)
+			(at 193.04 102.87 0)
 			(effects
 				(font
@@
 		)
 		(property "Description" "Power symbol creates a global label with name \"GNDD\" , digital ground"
-			(at 189.23 102.87 0)
+			(at 193.04 102.87 0)
 			(effects
 				(font
@@
 	(symbol
 		(lib_id "Power_Protection:USBLC6-2SC6")
-		(at 189.23 91.44 0)
+		(at 193.04 91.44 0)
 		(mirror y)
 		(unit 1)
@@
 		(dnp no)
 		(property "Reference" "U3"
-			(at 187.5789 83.82 0)
+			(at 191.3889 83.82 0)
 			(effects
 				(font
@@
 		)
 		(property "Value" "USBLC6-2SC6"
-			(at 187.5789 86.36 0)
+			(at 191.3889 86.36 0)
 			(effects
 				(font
@@
 		)
 		(property "Footprint" "Package_TO_SOT_SMD:SOT-23-6"
-			(at 187.96 97.79 0)
+			(at 191.77 97.79 0)
 			(effects
 				(font
@@
 		)
 		(property "Datasheet" "https://www.st.com/resource/en/datasheet/usblc6-2.pdf"
-			(at 187.96 99.695 0)
+			(at 191.77 99.695 0)
 			(effects
 				(font
@@
 		)
 		(property "Description" "Very low capacitance ESD protection diode, 2 data-line, SOT-23-6"
-			(at 189.23 91.44 0)
+			(at 193.04 91.44 0)
 			(effects
 				(font
@@
 	(symbol
 		(lib_id "power:+5V")
-		(at 189.23 81.28 0)
+		(at 193.04 81.28 0)
 		(unit 1)
 		(exclude_from_sim no)
@@
 		(dnp no)
 		(property "Reference" "#PWR017"
-			(at 189.23 85.09 0)
+			(at 193.04 85.09 0)
 			(effects
 				(font
@@
 		)
 		(property "Value" "+5V"
-			(at 186.436 78.994 0)
+			(at 190.246 78.994 0)
 			(effects
 				(font
@@
 		)
 		(property "Footprint" ""
-			(at 189.23 81.28 0)
+			(at 193.04 81.28 0)
 			(effects
 				(font
@@
 		)
 		(property "Datasheet" ""
-			(at 189.23 81.28 0)
+			(at 193.04 81.28 0)
 			(effects
 				(font
@@
 		)
 		(property "Description" "Power symbol creates a global label with name \"+5V\""
-			(at 189.23 81.28 0)
-			(effects
-				(font
+			(at 193.04 81.28 0)
+			(effects
+				(font

Commit message: Ningun cambio
Other:
- note added: "PROTECCION ESD"
- note removed: "PROTECCION EDS"
Changed lines of the file:
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@@
 	(generator_version "9.0")
 	(paper "A4")
-	(text "PROTECCION EDS"
+	(text "PROTECCION ESD"
 		(exclude_from_sim no)
 		(at 182.88 110.236 0)
