File: Hardware/Placa_PCB/Ground_Station.kicad_pcb (KiCad board)
At the start: 2 copper layers, 67.4 x 42.8 mm, 30 parts, among them J1 USB_C_Receptacle_USB2.0_16P, J2 Conn_01x08_Pin, J3 Conn_01x08_Pin, SW1 RESET, SW2 BOOT, U1 Ai-Thinker-Ra-02, U2 ESP32-S3-WROOM-1, U3 USBLC6-2SC6, U4 MIC29302AWD

Commit message: Agregando el PCB terminado
Parts:
- added G***: LOGO, Images:Logo_5x5, F.Cu at (128.7, 123.5)
- moved D2 57.1 mm to (145.3, 98.3), turned to 180 degrees
- moved R5 51.6 mm to (140.6, 98.3)
- moved C7 42.2 mm to (171.3, 91.3)
- moved R4 42.2 mm to (171.3, 87.9)
- moved R1 41.9 mm to (121.5, 116.5)
- moved C2 41.9 mm to (170.3, 122.1)
- moved C5 41.9 mm to (133.9, 101.9)
- moved J1 41.9 mm to (121.7, 104.9)
- moved R6 41.9 mm to (170.9, 96.5)
- moved R8 41.9 mm to (126.9, 116.5)
- moved U3 41.9 mm to (130.3, 104.9)
- moved C3 41.9 mm to (124.5, 93.1)
- moved C4 41.9 mm to (129.1, 99.9)
- moved R2 41.9 mm to (121.5, 113.1)
- moved C1 41.9 mm to (170.3, 119.3)
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Connections:
- J2 pad 2: +5V -> /MCU/3
- J2 pad 3: +3.3V -> /MCU/4
- J2 pad 4: /MCU/3 -> /MCU/5
- J2 pad 5: /MCU/4 -> /MCU/6
- J2 pad 6: /MCU/5 -> /MCU/7
- J2 pad 7: /MCU/6 -> /MCU/8
- J2 pad 8: /MCU/7 -> /MCU/21 - LED
- J3 pad 1: /MCU/8 -> +5V
- J3 pad 2: /MCU/15 -> +5V
- J3 pad 3: /MCU/16 -> +3.3V
- J3 pad 4: /MCU/17 -> +3.3V
- J3 pad 5: /MCU/18 -> GNDD
- J3 pad 6: /MCU/21 - LED -> GNDD
- R5 pad 1: +5V -> +3.3V
- U2 pad 10: /MCU/17 -> unconnected-(U2-IO17-Pad10)
- U2 pad 11: /MCU/18 -> unconnected-(U2-IO18-Pad11)
- U2 pad 8: /MCU/15 -> unconnected-(U2-IO15-Pad8)
- U2 pad 9: /MCU/16 -> unconnected-(U2-IO16-Pad9)
- U3 pad 1: /Alimentacion + USB/USB_D- -> /Alimentacion + USB/D-
- U3 pad 3: /Alimentacion + USB/USB_D+ -> /Alimentacion + USB/D+
- U3 pad 4: /Alimentacion + USB/D+ -> /Alimentacion + USB/USB_D+
- U3 pad 6: /Alimentacion + USB/D- -> /Alimentacion + USB/USB_D-
Routing:
- net GNDD: track 0.00 -> 60.6 mm, vias 0 -> 166
- net /MCU/7: track 0.00 -> 47.8 mm, vias 0 -> 2
- net /MCU/6: track 0.00 -> 46.7 mm, vias 0 -> 2
- net /MCU/5: track 0.00 -> 45.7 mm, vias 0 -> 2
- net /MCU/21 - LED: track 0.00 -> 44.6 mm, vias 0 -> 2
- net /MCU/4: track 0.00 -> 44.5 mm, vias 0 -> 2
- net /MCU/8: track 0.00 -> 37.8 mm, vias 0 -> 2
- net /MCU/BOOT: track 0.00 -> 34.2 mm, vias 0 -> 4
- net +5V: track 0.00 -> 33.9 mm, vias 0 -> 12
- net /MCU/3: track 0.00 -> 28.1 mm, vias 0 -> 2
- net /MCU/Tx: track 0.00 -> 24.2 mm, vias 0 -> 2
- net /MCU/EN: track 0.00 -> 23.0 mm, vias 0 -> 2
- net /LoRa/NSS': track 0.00 -> 22.8 mm
- net /MCU/Rx: track 0.00 -> 22.2 mm, vias 0 -> 2
- net /Alimentacion + USB/USB_D-: track 0.00 -> 20.0 mm
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- added copper zone on F.Cu, net +3.3V
- added copper zone on B.Cu, net +5V
- added copper zone on In1.Cu, net GNDD
- added copper zone on In2.Cu, net GNDD
Other:
- copper layers 2 -> 4
- board text added: "+3.3V"
- board text added: "+5V"
- board text added: "-"
- board text added: "D21"
- board text added: "D3"
- board text added: "D4"
- board text added: "D5"
- board text added: "D6"
- board text added: "D7"
- board text added: "D8"
- board text added: "Esteban Ruiz José Medina"
- board text added: "Frecuency: 433 MHz"
- board text added: "GND"
- board text added: "GROUND STATION - IIS FIUNA"
- board text added: "RX"
- board text added: "TX"
- board text added: "| |"
- board text removed: "Esteban Ruiz - José Medina"
- board text removed: "GROUND STATION - IIS"

Commit message: Placa Final
Routing:
- net +3.3V: track 6.68 -> 180.7 mm, vias 11 -> 7
- net +5V: track 33.9 -> 121.5 mm, vias 12 -> 4
- net GNDD: track 60.6 -> 32.0 mm, vias 166 -> 106
- net /MCU/21 - LED: track 44.6 -> 44.0 mm, vias 2 -> 1
- net /MCU/8: track 37.8 -> 38.0 mm, vias 2 -> 1
- net /MCU/4: track 44.5 -> 44.6 mm, vias 2 -> 1
- net /MCU/7: vias 2 -> 1
- net /MCU/6: vias 2 -> 1
- net /MCU/5: vias 2 -> 1
- added copper zone on B.Cu, net GNDD
- added copper zone on F.Cu, net GNDD
- removed copper zone on F.Cu, net +3.3V
- removed copper zone on B.Cu, net +5V

Commit message: Actualizacion PCB
Routing:
- net GNDD: vias 106 -> 112
Changed lines of the file:
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@@
 			(outputformat 1)
 			(mirror no)
-			(drillshape 1)
+			(drillshape 0)
 			(scaleselection 1)
-			(outputdirectory "")
+			(outputdirectory "../Gerbers/")
 		)
 	)
@@
 		)
 	)
+	(dimension
+		(type orthogonal)
+		(layer "F.Cu")
+		(pts
+			(xy 119.25 127.1) (xy 186.665 127.1)
+		)
+		(height 4.63)
+		(orientation 0)
+		(format
+			(prefix "")
+			(suffix "")
+			(units 3)
+			(units_format 0)
+			(precision 4)
+			(suppress_zeroes yes)
+		)
+		(style
+			(thickness 0.2)
+			(arrow_length 1.27)
+			(text_position_mode 0)
+			(arrow_direction outward)
+			(extension_height 0.58642)
+			(extension_offset 0.5)
+			(keep_text_aligned yes)
+		)
+		(gr_text "67.415"
+			(at 152.9575 129.93 0)
+			(layer "F.Cu")
+			(effects
+				(font
+					(size 1.5 1.5)
+					(thickness 0.3)
+				)
+			)
+		)
+	)
+	(dimension
+		(type orthogonal)
+		(layer "F.Cu")
+		(pts
+			(xy 186.665 127.1) (xy 186.665 84.3)
+		)
+		(height 3.345)
+		(orientation 1)
+		(format
+			(prefix "")
+			(suffix "")
+			(units 3)
+			(units_format 0)
+			(precision 4)
+			(suppress_zeroes yes)
+		)
+		(style
+			(thickness 0.2)
+			(arrow_length 1.27)
+			(text_position_mode 0)
+			(arrow_direction outward)
+			(extension_height 0.58642)
+			(extension_offset 0.5)
+			(keep_text_aligned yes)
+		)
+		(gr_text "42.8"
+			(at 188.21 105.7 90)
+			(layer "F.Cu")
+			(effects
+				(font
+					(size 1.5 1.5)
+					(thickness 0.3)
+				)
+			)
+		)
+	)
 	(segment
 		(start 170.35 86.25)
@@
 	)
 	(via
+		(at 185.51 121.31)
+		(size 0.6)
+		(drill 0.3)
+		(layers "F.Cu" "B.Cu")
+		(free yes)
+		(net 2)
+	)
+	(via
 		(at 151.525 91.375)
 		(size 0.6)
@@
 	)
 	(via
+		(at 185.48 97.92)
+		(size 0.6)
+		(drill 0.3)
+		(layers "F.Cu" "B.Cu")
+		(free yes)
+		(net 2)
+	)
+	(via
 		(at 161.53 118.44)
 		(size 0.6)
@@
 	)
 	(via
+		(at 179.88 108.58)
+		(size 0.6)
+		(drill 0.3)
+		(layers "F.Cu" "B.Cu")
+		(free yes)
+		(net 2)
+	)
+	(via
 		(at 132.25 116.95)
 		(size 0.6)
@@
 	)
 	(via
+		(at 185.48 103.58)
+		(size 0.6)
+		(drill 0.3)
+		(layers "F.Cu" "B.Cu")
+		(free yes)
+		(net 2)
+	)
+	(via
 		(at 175.57 85.99)
 		(size 0.6)
@@
 	)
 	(via
+		(at 185.39 114.98)
+		(size 0.6)
+		(drill 0.3)
+		(layers "F.Cu" "B.Cu")
+		(free yes)
+		(net 2)
+	)
+	(via
 		(at 134.12 91.51)
 		(size 0.6)
@@
 		(size 0.6)
 		(drill 0.3)
+		(layers "F.Cu" "B.Cu")
+		(free yes)
+		(net 2)
+	)
+	(via
+		(at 185.42 109.06)
+		(size 0.6)
+		(drill 0.3)
